File: StreamBoy_v0.1/StreamBoy.sch (KiCad schematic (older format))
At the start: 1 part

Commit message: Bunch of stuff
Parts:
- removed H1: MountingHole, footprints:ArtBender, symbol Mechanical:MountingHole
Connections:
- net labels removed: ESP_DAC1, GB_VIN
- wire segments 1 -> 0
Other:
- note removed: "For next revision:\nFix esp spacing\nExpose reset to fpga\n"
Changed lines of the file:
@@
 Comment4 ""
 $EndDescr
-$Comp
-L Mechanical:MountingHole H1
-U 1 1 5D2E04C3
-P 10550 6350
-F 0 "H1" H 10650 6396 50  0000 L CNN
-F 1 "MountingHole" H 10650 6305 50  0000 L CNN
-F 2 "footprints:ArtBender" H 10550 6350 50  0001 C CNN
-F 3 "~" H 10550 6350 50  0001 C CNN
-	1    10550 6350
-	1    0    0    -1
-$EndComp
-Text GLabel 3650 4150 0    50   Input ~ 0
-ESP_DAC1
-Text GLabel 3950 4150 2    50   Input ~ 0
-GB_VIN
-Wire Wire Line
-	3650 4150 3950 4150
-Text Notes 2550 5850 0    118  ~ 0
-For next revision:\nFix esp spacing\nExpose reset to fpga\n
 $Sheet
 S 2850 800  1250 800
@@
 $EndSheet
 $Sheet
-S 4800 2600 750  550
-U 5E087685
-F0 "Headers" 50
-F1 "Headers.sch" 50
+S 1150 3500 550  550
+U 5E07E0B7
+F0 "Misc" 50
+F1 "Misc.sch" 50
 $EndSheet
 $Sheet
-S 1150 3500 550  550
-U 5E07E0B7
-F0 "USB" 50
-F1 "USB.sch" 50
+S 8150 1300 2400 2100
+U 5E087685
+F0 "Debug" 50
+F1 "Debug.sch" 50
 $EndSheet
 $EndSCHEMATC
