File: StreamBoy_v0.1/Misc.sch (KiCad schematic (older format))
At the start: 12 parts, among them IC1 LY68L6400SLIT, U12 CP2102N-A01-GQFN28, X1 SG-7050CBN

Commit message: GB Reset fixed and moved some stuff
Parts:
- added C?: 0.01uf, Capacitor_SMD:C_0402_1005Metric, symbol Device:C
- added IC?: 6N137S1(TA), 6N137S1-TA:SOIC-8, symbol 6N137S1-TA:6N137S1(TA)
- added R?: 270Ohm, Capacitor_SMD:C_0603_1608Metric, symbol Device:R
- C9: lcscPartnum (none) -> C23733
Connections:
- net labels added: 5VCC, ESP_GB_RESET, GB_RSTN
- wire segments 45 -> 52
Changed lines of the file:
@@
 F 2 "Capacitor_SMD:C_0402_1005Metric" H 3538 1050 50  0001 C CNN
 F 3 "~" H 3500 1200 50  0001 C CNN
+F 4 "C23733" H 3500 1200 50  0001 C CNN "lcscPartnum"
 	1    3500 1200
 	-1   0    0    1
@@
 	0    1    1    0
 $EndComp
+$Comp
+L 6N137S1-TA:6N137S1(TA) IC?
+U 1 1 5E4AE392
+P 7750 5000
+F 0 "IC?" H 7475 5675 50  0000 C CNN
+F 1 "6N137S1(TA)" H 7475 5584 50  0000 C CNN
+F 2 "6N137S1-TA:SOIC-8" H 7750 5000 50  0001 C CNN
+F 3 "https://datasheet.lcsc.com/szlcsc/1908282202_Everlight-Elec-6N137S1-TA_C110020.pdf" H 7750 5000 50  0001 C CNN
+F 4 "C110020" H 7750 5000 50  0001 C CNN "lcscPartnum"
+	1    7750 5000
+	1    0    0    -1
+$EndComp
+Text GLabel 7850 4550 2    50   Input ~ 0
+5VCC
+Text GLabel 8650 4650 2    50   Input ~ 0
+5VCC
+Text GLabel 7850 4750 2    50   Input ~ 0
+GB_RSTN
+$Comp
+L power:GND #PWR?
+U 1 1 5E4AE39B
+P 8500 5050
+F 0 "#PWR?" H 8500 4800 50  0001 C CNN
+F 1 "GND" H 8505 4877 50  0000 C CNN
+F 2 "" H 8500 5050 50  0001 C CNN
+F 3 "" H 8500 5050 50  0001 C CNN
+	1    8500 5050
+	1    0    0    -1
+$EndComp
+$Comp
+L power:GND #PWR?
+U 1 1 5E4AE3A1
+P 7100 4750
+F 0 "#PWR?" H 7100 4500 50  0001 C CNN
+F 1 "GND" V 7105 4622 50  0000 R CNN
+F 2 "" H 7100 4750 50  0001 C CNN
+F 3 "" H 7100 4750 50  0001 C CNN
+	1    7100 4750
+	0    1    1    0
+$EndComp
+Wire Wire Line
+	8650 4650 8500 4650
+Wire Wire Line
+	8500 4700 8500 4650
+Connection ~ 8500 4650
+Wire Wire Line
+	8500 4650 7850 4650
+Wire Wire Line
+	7850 4850 8200 4850
+Wire Wire Line
+	8500 5000 8200 5000
+Wire Wire Line
+	8200 4850 8200 5000
+Wire Wire Line
+	8500 5000 8500 5050
+$Comp
+L Device:C C?
+U 1 1 5E4AE3AF
+P 8500 4850
+F 0 "C?" H 8615 4896 50  0000 L CNN
+F 1 "0.01uf" H 8615 4805 50  0000 L CNN
+F 2 "Capacitor_SMD:C_0402_1005Metric" H 8538 4700 50  0001 C CNN
+F 3 "~" H 8500 4850 50  0001 C CNN
+	1    8500 4850
+	1    0    0    -1
+$EndComp
+Connection ~ 8500 5000
+$Comp
+L Device:R R?
+U 1 1 5E4AE3B7
+P 6950 4650
+F 0 "R?" V 6743 4650 50  0000 C CNN
+F 1 "270Ohm" V 6834 4650 50  0000 C CNN
+F 2 "Capacitor_SMD:C_0603_1608Metric" V 6880 4650 50  0001 C CNN
+F 3 "~" H 6950 4650 50  0001 C CNN
+F 4 "C22966" H 6950 4650 50  0001 C CNN "lcscPartnum"
+	1    6950 4650
+	0    1    1    0
+$EndComp
+Text GLabel 6800 4650 0    50   Input ~ 0
+ESP_GB_RESET
 $EndSCHEMATC
